Commit message: Add Gazebo support. Changed joint limits.

File: onrobot_description/urdf/onrobot_rg.urdf.xacro (robot description, xacro)
@@ -3,6 +3,12 @@
   <!-- materials -->
   <xacro:include filename="$(find onrobot_description)/urdf/materials.urdf.xacro" />
+  <!-- transmission -->
+  <xacro:include filename="$(find onrobot_description)/urdf/onrobot_rg.transmission.xacro" />
+  <!-- gazebo -->
+  <xacro:include filename="$(find onrobot_description)/urdf/onrobot_rg.gazebo.xacro" />
   <!-- onrobot gripper -->
-  <xacro:macro name="onrobot_rg" params="parent *origin prefix:='gripper' model:='rg2_v1' safety_shield:=False bracket:='single_bracket' mount_angle:=0.0">
+  <xacro:macro name="onrobot_rg" params="parent *origin prefix:='gripper'
+    model:='rg2_v1' safety_shield:=False bracket:='single_bracket' mount_angle:=0.0
+    transmission_hw_interface:=hardware_interface/EffortJointInterface">
     <!-- load config from file -->
     <xacro:property name="config_file" value="$(find onrobot_description)/config/${model}.yaml"/>
@@ -11,9 +17,4 @@
     <xacro:property name="origin" value="${config['origin']}"/>
     <xacro:property name="limit" value="${config['limit']}"/>
-    <!-- joint helper -->
-    <xacro:macro name="joint_config" params="name">
-      <origin xyz="${origin[name]['x']} ${origin[name]['y']} ${origin[name]['z']}" rpy="0.0 0.0 0.0"/>
-      <limit lower="${limit['lower']}" upper="${limit['upper']}" effort="${limit['effort']}" velocity="${limit['velocity']}"/>
-    </xacro:macro>
     <!-- bracket -->
     <link name="${prefix}_bracket">
@@ -62,22 +63,13 @@
       <origin xyz="${origin[bracket]['x']} ${origin[bracket]['y']} ${origin[bracket]['z']}" rpy="${mount_angle} 0.0 0.0"/>
     </joint>
-    <!-- dummy motor link -->
-    <link name="${prefix}_motor">
-      <inertial>
-        <mass value="0.001"/>
-        <inertia ixx="0.001" iyy="0.001" izz="0.001" ixy="0.0" ixz="0.0" iyz="0.0"/>
-      </inertial>
-    </link>
-    <joint name="${prefix}_joint" type="revolute">
-      <parent link="${prefix}_body"/>
-      <child link = "${prefix}_motor"/>
-      <axis xyz="0 1 0"/>
-      <limit lower="0.0" upper="${limit['upper']-limit['lower']}" effort="${limit['effort']}" velocity="${limit['velocity']}"/>
-      <dynamics damping="0" friction="0"/>
-    </joint>
     <!-- fingers -->
     <xacro:macro name="finger" params="name is_master">
       <!-- origin -->
-      <link name="${name}_origin"/>
+      <link name="${name}_origin">
+        <inertial>
+          <mass value="0.001"/>
+          <inertia ixx="0.001" iyy="0.001" izz="0.001" ixy="0.0" ixz="0.0" iyz="0.0"/>
+        </inertial>
+      </link>
       <joint name="${name}_origin_joint" type="fixed">
         <parent link="${prefix}_body"/>
@@ -85,4 +77,33 @@
         <origin xyz="0 0 0" rpy="0 0 ${0 if is_master else pi}"/>
       </joint>
+      <!-- moment bar -->
+      <link name="${name}_moment_arm">
+        <visual>
+          <geometry>
+            <mesh filename="package://onrobot_description/meshes/${model}/visual/moment_arm.stl"/>
+          </geometry>
+          <material name="onrobot/light_grey"/>
+        </visual>
+        <collision>
+          <geometry>
+            <mesh filename="package://onrobot_description/meshes/${model}/collision/moment_arm.stl"/>
+          </geometry>
+        </collision>
+        <inertial>
+          <mass value="0.001"/>
+          <inertia ixx="0.001" iyy="0.001" izz="0.001" ixy="0.0" ixz="0.0" iyz="0.0"/>
+        </inertial>
+      </link>
+      <joint name="${prefix + ('' if is_master else '_mirror')}_joint" type="revolute">
+        <parent link="${name}_origin"/>
+        <child link = "${name}_moment_arm"/>
+        <axis xyz="0 1 0"/>
+        <origin xyz="${origin['moment_arm']['x']} ${origin['moment_arm']['y']} ${origin['moment_arm']['z']}" rpy="0.0 ${limit['offset']} 0.0"/>
+        <limit lower="${limit['lower']}" upper="${limit['upper']}" effort="${limit['effort']}" velocity="${limit['velocity']}"/>
+        <dynamics damping="0.1" friction="0.1"/>
+        <xacro:unless value="${is_master}">
+          <mimic joint="${prefix}_joint" multiplier="1" offset="0"/>
+        </xacro:unless>
+      </joint>
       <!-- truss bar -->
       <link name="${name}_truss_arm">
@@ -103,91 +124,12 @@
         </inertial>
       </link>
-      <joint name="${name}_joint" type="revolute">
+      <joint name="${name}_truss_arm_joint" type="revolute">
         <parent link="${name}_origin"/>
         <child link = "${name}_truss_arm"/>
         <axis xyz="0 1 0"/>
-        <xacro:joint_config name="truss_arm"/>
-        <mimic joint="${prefix}_joint" multiplier="-1" offset="${limit['upper']}"/>
-        <dynamics damping="0" friction="0"/>
-      </joint>
-      <!-- moment bar -->
-      <link name="${name}_moment_arm">
-        <visual>
-          <geometry>
-            <mesh filename="package://onrobot_description/meshes/${model}/visual/moment_arm.stl"/>
-          </geometry>
-          <material name="onrobot/light_grey"/>
-        </visual>
-        <collision>
-          <geometry>
-            <mesh filename="package://onrobot_description/meshes/${model}/collision/moment_arm.stl"/>
-          </geometry>
-        </collision>
-        <inertial>
-          <mass value="0.001"/>
-          <inertia ixx="0.001" iyy="0.001" izz="0.001" ixy="0.0" ixz="0.0" iyz="0.0"/>
-        </inertial>
-      </link>
-      <joint name="${name}_moment_arm_joint" type="revolute">
-        <parent link="${name}_origin"/>
-        <child link = "${name}_moment_arm"/>
-        <axis xyz="0 1 0"/>
-        <xacro:joint_config name="moment_arm"/>
-        <mimic joint="${prefix}_joint" multiplier="-1" offset="${limit['upper']}"/>
-        <dynamics damping="0" friction="0"/>
-      </joint>
-      <!-- finger tip -->
-      <link name="${name}_finger_tip">
-        <visual>
-          <geometry>
-            <mesh filename="package://onrobot_description/meshes/${model}/visual/finger_tip.stl"/>
-          </geometry>
-          <material name="onrobot/light_grey"/>
-        </visual>
-        <collision>
-          <geometry>
-            <mesh filename="package://onrobot_description/meshes/${model}/collision/finger_tip_1.stl"/>
-          </geometry>
-        </collision>
-        <collision>
-          <geometry>
-            <mesh filename="package://onrobot_description/meshes/${model}/collision/finger_tip_2.stl"/>
-          </geometry>
-        </collision>
-        <inertial>
-          <mass value="0.001"/>
-          <inertia ixx="0.001" iyy="0.001" izz="0.001" ixy="0.0" ixz="0.0" iyz="0.0"/>
-        </inertial>
-      </link>
-      <joint name="${name}_finger_tip_joint" type="revolute">
-        <parent link = "${name}_truss_arm"/>
-        <child link = "${name}_finger_tip"/>
-        <axis xyz="0 -1 0"/>
-        <xacro:joint_config name="finger_tip"/>
-        <mimic joint="${prefix}_joint" multiplier="-1" offset="${limit['upper']}"/>
-        <dynamics damping="0" friction="0"/>
-      </joint>
-      <!-- flex finger -->
-      <link name="${name}_flex_finger">
-        <visual>
-          <geometry>
-            <mesh filename="package://onrobot_description/meshes/${model}/visual/flex_finger.stl"/>
-          </geometry>
-          <material name="onrobot/dark_grey"/>
-        </visual>
-        <collision>
-          <geometry>
-            <mesh filename="package://onrobot_description/meshes/${model}/collision/flex_finger.stl"/>
-          </geometry>
-        </collision>
-        <inertial>
-          <mass value="0.001"/>
-          <inertia ixx="0.001" iyy="0.001" izz="0.001" ixy="0.0" ixz="0.0" iyz="0.0"/>
-        </inertial>
-      </link>
-      <joint name="${name}_flex_finger_joint" type="fixed">
-        <parent link="${name}_finger_tip"/>
-        <child link = "${name}_flex_finger"/>
-        <xacro:joint_config name="flex_finger"/>
+        <origin xyz="${origin['truss_arm']['x']} ${origin['truss_arm']['y']} ${origin['truss_arm']['z']}" rpy="0.0 ${limit['offset']} 0.0"/>
+        <limit lower="${limit['lower']}" upper="${limit['upper']}" effort="${limit['effort']}" velocity="${limit['velocity']}"/>
+        <dynamics damping="0.1" friction="0.1"/>
+        <mimic joint="${prefix}_joint" multiplier="1" offset="0"/>
       </joint>
       <!-- safety shield -->
@@ -200,9 +142,9 @@
             <material name="onrobot/dark_grey"/>
           </visual>
-          <collision>
+          <!-- <collision>
             <geometry>
               <mesh filename="package://onrobot_description/meshes/${model}/collision/safety_shield.stl"/>
             </geometry>
-          </collision>
+          </collision> -->
           <inertial>
             <mass value="0.001"/>
@@ -214,12 +156,70 @@
           <child link = "${name}_safety_shield"/>
           <axis xyz="0 1 0"/>
-          <xacro:joint_config name="safety_shield"/>
-          <mimic joint="${prefix}_joint" multiplier="-1" offset="${limit['upper']}"/>
-          <dynamics damping="0" friction="0"/>
+          <origin xyz="${origin['safety_shield']['x']} ${origin['safety_shield']['y']} ${origin['safety_shield']['z']}" rpy="0.0 ${limit['offset']} 0.0"/>
+          <limit lower="${limit['lower']}" upper="${limit['upper']}" effort="${limit['effort']}" velocity="${limit['velocity']}"/>
+          <dynamics damping="0.1" friction="0.1"/>
+          <mimic joint="${prefix}_joint" multiplier="1" offset="0"/>
         </joint>
       </xacro:if>
+      <!-- finger tip -->
+      <link name="${name}_finger_tip">
+        <visual>
+          <geometry>
+            <mesh filename="package://onrobot_description/meshes/${model}/visual/finger_tip.stl"/>
+          </geometry>
+          <material name="onrobot/light_grey"/>
+        </visual>
+        <collision>
+          <geometry>
+            <mesh filename="package://onrobot_description/meshes/${model}/collision/finger_tip_1.stl"/>
+          </geometry>
+        </collision>
+        <collision>
+          <geometry>
+            <mesh filename="package://onrobot_description/meshes/${model}/collision/finger_tip_2.stl"/>
+          </geometry>
+        </collision>
+        <inertial>
+          <mass value="0.001"/>
+          <inertia ixx="0.001" iyy="0.001" izz="0.001" ixy="0.0" ixz="0.0" iyz="0.0"/>
+        </inertial>
+      </link>
+      <joint name="${name}_finger_tip_joint" type="revolute">
+        <parent link = "${name}_truss_arm"/>
+        <child link = "${name}_finger_tip"/>
+        <axis xyz="0 -1 0"/>
+        <origin xyz="${origin['finger_tip']['x']} ${origin['finger_tip']['y']} ${origin['finger_tip']['z']}" rpy="0.0 ${-limit['offset']} 0.0"/>
+        <limit lower="${limit['lower']}" upper="${limit['upper']}" effort="${limit['effort']}" velocity="${limit['velocity']}"/>
+        <dynamics damping="0.1" friction="0.1"/>
+        <mimic joint="${prefix}_joint" multiplier="1" offset="0"/>
+      </joint>
+      <!-- flex finger -->
+      <link name="${name}_flex_finger">
+        <visual>
+          <geometry>
+            <mesh filename="package://onrobot_description/meshes/${model}/visual/flex_finger.stl"/>
+          </geometry>
+          <material name="onrobot/dark_grey"/>
+        </visual>
+        <collision>
+          <geometry>
+            <mesh filename="package://onrobot_description/meshes/${model}/collision/flex_finger.stl"/>
+          </geometry>
+        </collision>
+        <inertial>
+          <mass value="0.001"/>
+          <inertia ixx="0.001" iyy="0.001" izz="0.001" ixy="0.0" ixz="0.0" iyz="0.0"/>
+        </inertial>
+      </link>
+      <joint name="${name}_flex_finger_joint" type="fixed">
+        <parent link="${name}_finger_tip"/>
+        <child link = "${name}_flex_finger"/>
+        <origin xyz="${origin['flex_finger']['x']} ${origin['flex_finger']['y']} ${origin['flex_finger']['z']}" rpy="0.0 0.0 0.0"/>
+      </joint>
     </xacro:macro>
     <xacro:finger name="${prefix}_finger_1" is_master="true"/>
     <xacro:finger name="${prefix}_finger_2" is_master="false"/>
+    <xacro:rg_transmission prefix="${prefix}" hw_interface="${transmission_hw_interface}"/>
+    <xacro:rg_gazebo prefix="${prefix}" origin="${origin}" limit="${limit}" safety_shield="${safety_shield}"/>
   </xacro:macro>
 </robot>

Commit message: Add the grasp frame. Remove collision for the safety_shield link

File: onrobot_description/urdf/onrobot_rg.urdf.xacro (robot description, xacro)
@@ -63,4 +63,11 @@
       <origin xyz="${origin[bracket]['x']} ${origin[bracket]['y']} ${origin[bracket]['z']}" rpy="${mount_angle} 0.0 0.0"/>
     </joint>
+    <!-- grasp frame -->
+    <link name="${prefix}_grasp_frame"/>
+    <joint name="${prefix}_grasp_frame_joint" type="fixed">
+      <parent link="${prefix}_body"/>
+      <child link = "${prefix}_grasp_frame"/>
+      <origin xyz="${origin['grasp_frame']['x']} ${origin['grasp_frame']['y']} ${origin['grasp_frame']['z']}" rpy="0.0 0.0 0.0"/>
+    </joint>
     <!-- fingers -->
     <xacro:macro name="finger" params="name is_master">
@@ -142,9 +149,10 @@
             <material name="onrobot/dark_grey"/>
           </visual>
-          <!-- <collision>
+          <collision>
             <geometry>
-              <mesh filename="package://onrobot_description/meshes/${model}/collision/safety_shield.stl"/>
+              <!-- <mesh filename="package://onrobot_description/meshes/${model}/collision/safety_shield.stl"/> -->
+              <box size="0.0 0.0 0.0"/>
             </geometry>
-          </collision> -->
+          </collision>
           <inertial>
             <mass value="0.001"/>

Commit message: Optimize the description xacro

File: onrobot_description/urdf/onrobot_rg.urdf.xacro (robot description, xacro)
@@ -17,4 +17,10 @@
     <xacro:property name="origin" value="${config['origin']}"/>
     <xacro:property name="limit" value="${config['limit']}"/>
+    <xacro:macro name="_limit" params="">
+      <limit lower="${limit['lower']}" upper="${limit['upper']}" effort="${limit['effort']}" velocity="${limit['velocity']}"/>
+    </xacro:macro>
+    <xacro:macro name="_frame" params="id rpy">
+      <origin xyz="${origin[id]['x']} ${origin[id]['y']} ${origin[id]['z']}" rpy="${rpy}"/>
+    </xacro:macro>
     <!-- bracket -->
     <link name="${prefix}_bracket">
@@ -61,5 +67,5 @@
       <parent link="${prefix}_bracket"/>
       <child link = "${prefix}_body"/>
-      <origin xyz="${origin[bracket]['x']} ${origin[bracket]['y']} ${origin[bracket]['z']}" rpy="${mount_angle} 0.0 0.0"/>
+      <xacro:_frame id="${bracket}" rpy="${mount_angle} 0.0 0.0"/>
     </joint>
     <!-- grasp frame -->
@@ -68,18 +74,18 @@
       <parent link="${prefix}_body"/>
       <child link = "${prefix}_grasp_frame"/>
-      <origin xyz="${origin['grasp_frame']['x']} ${origin['grasp_frame']['y']} ${origin['grasp_frame']['z']}" rpy="0.0 0.0 0.0"/>
+      <xacro:_frame id="grasp_frame" rpy="0.0 0.0 0.0"/>
     </joint>
     <!-- fingers -->
     <xacro:macro name="finger" params="name is_master">
       <!-- origin -->
-      <link name="${name}_origin">
-        <inertial>
-          <mass value="0.001"/>
-          <inertia ixx="0.001" iyy="0.001" izz="0.001" ixy="0.0" ixz="0.0" iyz="0.0"/>
-        </inertial>
-      </link>
-      <joint name="${name}_origin_joint" type="fixed">
+      <link name="${name}_frame">
+        <inertial>
+          <mass value="0.001"/>
+          <inertia ixx="0.001" iyy="0.001" izz="0.001" ixy="0.0" ixz="0.0" iyz="0.0"/>
+        </inertial>
+      </link>
+      <joint name="${name}_frame_joint" type="fixed">
         <parent link="${prefix}_body"/>
-        <child link = "${name}_origin"/>
+        <child link = "${name}_frame"/>
         <origin xyz="0 0 0" rpy="0 0 ${0 if is_master else pi}"/>
       </joint>
@@ -103,9 +109,9 @@
       </link>
       <joint name="${prefix + ('' if is_master else '_mirror')}_joint" type="revolute">
-        <parent link="${name}_origin"/>
+        <parent link="${name}_frame"/>
         <child link = "${name}_moment_arm"/>
         <axis xyz="0 1 0"/>
-        <origin xyz="${origin['moment_arm']['x']} ${origin['moment_arm']['y']} ${origin['moment_arm']['z']}" rpy="0.0 ${limit['offset']} 0.0"/>
-        <limit lower="${limit['lower']}" upper="${limit['upper']}" effort="${limit['effort']}" velocity="${limit['velocity']}"/>
+        <xacro:_frame id="moment_arm" rpy="0.0 ${limit['offset']} 0.0"/>
+        <xacro:_limit/>
         <dynamics damping="0.1" friction="0.1"/>
         <xacro:unless value="${is_master}">
@@ -132,9 +138,9 @@
       </link>
       <joint name="${name}_truss_arm_joint" type="revolute">
-        <parent link="${name}_origin"/>
+        <parent link="${name}_frame"/>
         <child link = "${name}_truss_arm"/>
         <axis xyz="0 1 0"/>
-        <origin xyz="${origin['truss_arm']['x']} ${origin['truss_arm']['y']} ${origin['truss_arm']['z']}" rpy="0.0 ${limit['offset']} 0.0"/>
-        <limit lower="${limit['lower']}" upper="${limit['upper']}" effort="${limit['effort']}" velocity="${limit['velocity']}"/>
+        <xacro:_frame id="truss_arm" rpy="0.0 ${limit['offset']} 0.0"/>
+        <xacro:_limit/>
         <dynamics damping="0.1" friction="0.1"/>
         <mimic joint="${prefix}_joint" multiplier="1" offset="0"/>
@@ -164,6 +170,6 @@
           <child link = "${name}_safety_shield"/>
           <axis xyz="0 1 0"/>
-          <origin xyz="${origin['safety_shield']['x']} ${origin['safety_shield']['y']} ${origin['safety_shield']['z']}" rpy="0.0 ${limit['offset']} 0.0"/>
-          <limit lower="${limit['lower']}" upper="${limit['upper']}" effort="${limit['effort']}" velocity="${limit['velocity']}"/>
+          <xacro:_frame id="safety_shield" rpy="0.0 ${limit['offset']} 0.0"/>
+          <xacro:_limit/>
           <dynamics damping="0.1" friction="0.1"/>
           <mimic joint="${prefix}_joint" multiplier="1" offset="0"/>
@@ -197,6 +203,6 @@
         <child link = "${name}_finger_tip"/>
         <axis xyz="0 -1 0"/>
-        <origin xyz="${origin['finger_tip']['x']} ${origin['finger_tip']['y']} ${origin['finger_tip']['z']}" rpy="0.0 ${-limit['offset']} 0.0"/>
-        <limit lower="${limit['lower']}" upper="${limit['upper']}" effort="${limit['effort']}" velocity="${limit['velocity']}"/>
+        <xacro:_frame id="finger_tip" rpy="0.0 ${-limit['offset']} 0.0"/>
+        <xacro:_limit/>
         <dynamics damping="0.1" friction="0.1"/>
         <mimic joint="${prefix}_joint" multiplier="1" offset="0"/>
@@ -223,5 +229,5 @@
         <parent link="${name}_finger_tip"/>
         <child link = "${name}_flex_finger"/>
-        <origin xyz="${origin['flex_finger']['x']} ${origin['flex_finger']['y']} ${origin['flex_finger']['z']}" rpy="0.0 0.0 0.0"/>
+        <xacro:_frame id="flex_finger" rpy="0.0 0.0 0.0"/>
       </joint>
     </xacro:macro>
