Commit message: Move inertial parameters to the config file

File: onrobot_description/urdf/onrobot_rg.urdf.xacro (robot description, xacro)
@@ -14,12 +14,20 @@
     <xacro:property name="config_file" value="$(find onrobot_description)/config/${model}.yaml"/>
     <xacro:property name="config" value="${load_yaml(config_file)}"/>
-    <xacro:property name="mass" value="${config['mass']}"/>
+    <xacro:property name="limit" value="${config['limit']}"/>
     <xacro:property name="origin" value="${config['origin']}"/>
-    <xacro:property name="limit" value="${config['limit']}"/>
+    <xacro:property name="inertial" value="${config['inertial']}"/>
     <xacro:macro name="_limit" params="">
-      <limit lower="${limit['lower']}" upper="${limit['upper']}" effort="${limit['effort']}" velocity="${limit['velocity']}"/>
+      <limit lower="${limit['lower']}" upper="${limit['upper']}"
+             effort="${limit['effort']}" velocity="${limit['velocity']}"/>
     </xacro:macro>
     <xacro:macro name="_frame" params="id rpy">
       <origin xyz="${origin[id]['x']} ${origin[id]['y']} ${origin[id]['z']}" rpy="${rpy}"/>
+    </xacro:macro>
+    <xacro:macro name="_inertial" params="id">
+      <inertial>
+        <mass value="${inertial[id]['mass']}"/>
+        <inertia ixx="${inertial[id]['ixx']}" iyy="${inertial[id]['iyy']}" izz="${inertial[id]['izz']}"
+                 ixy="${inertial[id]['ixy']}" ixz="${inertial[id]['ixz']}" iyz="${inertial[id]['iyz']}"/>
+      </inertial>
     </xacro:macro>
     <!-- bracket -->
@@ -36,8 +44,5 @@
         </geometry>
       </collision>
-      <inertial>
-        <mass value="0.001"/>
-        <inertia ixx="0.001" iyy="0.001" izz="0.001" ixy="0.0" ixz="0.0" iyz="0.0"/>
-      </inertial>
+      <xacro:_inertial id="${bracket}"/>
     </link>
     <joint name="${prefix}_bracket_joint" type="fixed">
@@ -59,8 +64,5 @@
         </geometry>
       </collision>
-      <inertial>
-        <mass value="${mass}"/>
-        <inertia ixx="0.001" iyy="0.001" izz="0.001" ixy="0.0" ixz="0.0" iyz="0.0"/>
-      </inertial>
+      <xacro:_inertial id="body"/>
     </link>
     <joint name="${prefix}_body_joint" type="fixed">
@@ -78,11 +80,6 @@
     <!-- fingers -->
     <xacro:macro name="finger" params="name is_master">
-      <!-- origin -->
-      <link name="${name}_frame">
-        <inertial>
-          <mass value="0.001"/>
-          <inertia ixx="0.001" iyy="0.001" izz="0.001" ixy="0.0" ixz="0.0" iyz="0.0"/>
-        </inertial>
-      </link>
+      <!-- origin frame -->
+      <link name="${name}_frame"/>
       <joint name="${name}_frame_joint" type="fixed">
         <parent link="${prefix}_body"/>
@@ -103,8 +100,5 @@
           </geometry>
         </collision>
-        <inertial>
-          <mass value="0.001"/>
-          <inertia ixx="0.001" iyy="0.001" izz="0.001" ixy="0.0" ixz="0.0" iyz="0.0"/>
-        </inertial>
+        <xacro:_inertial id="moment_arm"/>
       </link>
       <joint name="${prefix + ('' if is_master else '_mirror')}_joint" type="revolute">
@@ -132,8 +126,5 @@
           </geometry>
         </collision>
-        <inertial>
-          <mass value="0.001"/>
-          <inertia ixx="0.001" iyy="0.001" izz="0.001" ixy="0.0" ixz="0.0" iyz="0.0"/>
-        </inertial>
+        <xacro:_inertial id="truss_arm"/>
       </link>
       <joint name="${name}_truss_arm_joint" type="revolute">
@@ -161,8 +152,5 @@
             </geometry>
           </collision>
-          <inertial>
-            <mass value="0.001"/>
-            <inertia ixx="0.001" iyy="0.001" izz="0.001" ixy="0.0" ixz="0.0" iyz="0.0"/>
-          </inertial>
+          <xacro:_inertial id="safety_shield"/>
         </link>
         <joint name="${name}_safety_shield_joint" type="revolute">
@@ -194,8 +182,5 @@
           </geometry>
         </collision>
-        <inertial>
-          <mass value="0.001"/>
-          <inertia ixx="0.001" iyy="0.001" izz="0.001" ixy="0.0" ixz="0.0" iyz="0.0"/>
-        </inertial>
+        <xacro:_inertial id="finger_tip"/>
       </link>
       <joint name="${name}_finger_tip_joint" type="revolute">
@@ -221,8 +206,5 @@
           </geometry>
         </collision>
-        <inertial>
-          <mass value="0.001"/>
-          <inertia ixx="0.001" iyy="0.001" izz="0.001" ixy="0.0" ixz="0.0" iyz="0.0"/>
-        </inertial>
+        <xacro:_inertial id="flex_finger"/>
       </link>
       <joint name="${name}_flex_finger_joint" type="fixed">

Commit message: Move offset to the kinematics settings

File: onrobot_description/urdf/onrobot_rg.urdf.xacro (robot description, xacro)
@@ -17,4 +17,5 @@
     <xacro:property name="origin" value="${config['origin']}"/>
     <xacro:property name="inertial" value="${config['inertial']}"/>
+    <xacro:property name="offset" value="${config['kinematics']['offset']}"/>
     <xacro:macro name="_limit" params="">
       <limit lower="${limit['lower']}" upper="${limit['upper']}"
@@ -106,5 +107,5 @@
         <child link = "${name}_moment_arm"/>
         <axis xyz="0 1 0"/>
-        <xacro:_frame id="moment_arm" rpy="0.0 ${limit['offset']} 0.0"/>
+        <xacro:_frame id="moment_arm" rpy="0.0 ${offset} 0.0"/>
         <xacro:_limit/>
         <dynamics damping="0.1" friction="0.1"/>
@@ -132,5 +133,5 @@
         <child link = "${name}_truss_arm"/>
         <axis xyz="0 1 0"/>
-        <xacro:_frame id="truss_arm" rpy="0.0 ${limit['offset']} 0.0"/>
+        <xacro:_frame id="truss_arm" rpy="0.0 ${offset} 0.0"/>
         <xacro:_limit/>
         <dynamics damping="0.1" friction="0.1"/>
@@ -158,5 +159,5 @@
           <child link = "${name}_safety_shield"/>
           <axis xyz="0 1 0"/>
-          <xacro:_frame id="safety_shield" rpy="0.0 ${limit['offset']} 0.0"/>
+          <xacro:_frame id="safety_shield" rpy="0.0 ${offset} 0.0"/>
           <xacro:_limit/>
           <dynamics damping="0.1" friction="0.1"/>
@@ -188,5 +189,5 @@
         <child link = "${name}_finger_tip"/>
         <axis xyz="0 -1 0"/>
-        <xacro:_frame id="finger_tip" rpy="0.0 ${-limit['offset']} 0.0"/>
+        <xacro:_frame id="finger_tip" rpy="0.0 ${-offset} 0.0"/>
         <xacro:_limit/>
         <dynamics damping="0.1" friction="0.1"/>
