Commit message: Tune gripper description

File: onrobot_description/urdf/onrobot_rg.gazebo.xacro (robot description, xacro)
@@ -22,5 +22,5 @@
     </gazebo>
     <!-- enable mimic joints -->
-    <xacro:macro name="mimic_joint" params="name has_pid:=true max_effort:=40.0">
+    <xacro:macro name="mimic_joint" params="name has_pid:=true">
       <plugin name="${name}_mimic_joint_plugin" filename="libroboticsgroup_upatras_gazebo_mimic_joint_plugin.so">
         <joint>${prefix}_joint</joint>

File: onrobot_description/urdf/onrobot_rg.transmission.xacro (robot description, xacro)
@@ -1,5 +1,5 @@
 <?xml version="1.0"?>
 <robot xmlns:xacro="http://ros.org/wiki/xacro">
-  <xacro:macro name="rg_transmission" params="prefix hw_interface:='hardware_interface/EffortJointInterface'">
+  <xacro:macro name="rg_transmission" params="prefix hw_interface">
     <transmission name="${prefix}_joint_trans">
       <type>transmission_interface/SimpleTransmission</type>
@@ -8,4 +8,5 @@
       </joint>
       <actuator name="${prefix}_joint_motor">
+        <hardwareInterface>${hw_interface}</hardwareInterface>
         <mechanicalReduction>1</mechanicalReduction>
       </actuator>

File: onrobot_description/urdf/onrobot_rg.urdf.xacro (robot description, xacro)
@@ -82,8 +82,13 @@
     <xacro:macro name="finger" params="name is_master">
       <!-- origin frame -->
-      <link name="${name}_frame"/>
-      <joint name="${name}_frame_joint" type="fixed">
+      <link name="${name}_origin">
+        <inertial>
+          <mass value="0.001"/>
+          <inertia ixx="0.00001" ixy="0.0" ixz="0.0" iyy="0.00001" iyz="0.0" izz="0.00001"/>
+        </inertial>
+      </link>
+      <joint name="${name}_origin_joint" type="fixed">
         <parent link="${prefix}_body"/>
-        <child link = "${name}_frame"/>
+        <child link = "${name}_origin"/>
         <origin xyz="0 0 0" rpy="0 0 ${0 if is_master else pi}"/>
       </joint>
@@ -104,10 +109,10 @@
       </link>
       <joint name="${prefix + ('' if is_master else '_mirror')}_joint" type="revolute">
-        <parent link="${name}_frame"/>
+        <parent link="${name}_origin"/>
         <child link = "${name}_moment_arm"/>
         <axis xyz="0 1 0"/>
         <xacro:_frame id="moment_arm" rpy="0.0 ${offset} 0.0"/>
         <xacro:_limit/>
-        <dynamics damping="0.1" friction="0.1"/>
+        <dynamics damping="1" friction="0"/>
         <xacro:unless value="${is_master}">
           <mimic joint="${prefix}_joint" multiplier="1" offset="0"/>
@@ -130,10 +135,10 @@
       </link>
       <joint name="${name}_truss_arm_joint" type="revolute">
-        <parent link="${name}_frame"/>
+        <parent link="${name}_origin"/>
         <child link = "${name}_truss_arm"/>
         <axis xyz="0 1 0"/>
         <xacro:_frame id="truss_arm" rpy="0.0 ${offset} 0.0"/>
         <xacro:_limit/>
-        <dynamics damping="0.1" friction="0.1"/>
+        <dynamics damping="1" friction="1"/>
         <mimic joint="${prefix}_joint" multiplier="1" offset="0"/>
       </joint>
@@ -161,5 +166,5 @@
           <xacro:_frame id="safety_shield" rpy="0.0 ${offset} 0.0"/>
           <xacro:_limit/>
-          <dynamics damping="0.1" friction="0.1"/>
+          <dynamics damping="1" friction="1"/>
           <mimic joint="${prefix}_joint" multiplier="1" offset="0"/>
         </joint>
@@ -191,5 +196,5 @@
         <xacro:_frame id="finger_tip" rpy="0.0 ${-offset} 0.0"/>
         <xacro:_limit/>
-        <dynamics damping="0.1" friction="0.1"/>
+        <dynamics damping="1" friction="1"/>
         <mimic joint="${prefix}_joint" multiplier="1" offset="0"/>
       </joint>

Commit message: Switch from ros_control to dedicated gazebo plugin

File: onrobot_description/urdf/onrobot_rg.gazebo.xacro (robot description, xacro)
@@ -2,10 +2,26 @@
 <robot xmlns:xacro="http://ros.org/wiki/xacro">
   <xacro:macro name="rg_gazebo" params="prefix origin limit safety_shield:=False">
+    <!-- load "onrobot_gripper_plugin" plugin -->
+    <gazebo>
+      <plugin name="${prefix}_plugin" filename="libonrobot_gripper_plugin.so">
+        <robotNamespace>/${prefix}</robotNamespace>
+        <jointName>${prefix}_joint, ${prefix}_mirror_joint</jointName>
+        <tipName>${prefix}_finger_1_finger_tip, ${prefix}_finger_2_finger_tip</tipName>
+        <palmName>${prefix}_body</palmName>
+        <xacro:if value="${safety_shield}">
+          <mimicName>${prefix}_finger_1_safety_shield_joint, ${prefix}_finger_2_safety_shield_joint</mimicName>
+        </xacro:if>
+        <maxEffort>0.5</maxEffort>
+      </plugin>
+    </gazebo>
     <!-- add close loop joints -->
-    <xacro:macro name="close_loop_joint" params="name xyz">
+    <xacro:property name="x" value="${origin['moment_arm']['x']-origin['truss_arm']['x']}"/>
+    <xacro:property name="y" value="${origin['moment_arm']['y']-origin['truss_arm']['y']}"/>
+    <xacro:property name="z" value="${origin['moment_arm']['z']-origin['truss_arm']['z']}"/>
+    <xacro:macro name="close_loop_joint" params="name">
       <joint name='${name}_close_loop_joint' type='revolute'>
         <parent>${name}_moment_arm</parent>
         <child>${name}_finger_tip</child>
-        <pose frame=''>${xyz} 0 0 0</pose>
+        <pose frame=''>${x} ${y} ${z} 0 0 0</pose>
         <axis>
           <xyz>0 -1 0</xyz>
@@ -15,31 +31,30 @@
     </xacro:macro>
     <gazebo>
-      <xacro:property name="x" value="${origin['moment_arm']['x']-origin['truss_arm']['x']}"/>
-      <xacro:property name="y" value="${origin['moment_arm']['y']-origin['truss_arm']['y']}"/>
-      <xacro:property name="z" value="${origin['moment_arm']['z']-origin['truss_arm']['z']}"/>
-      <xacro:close_loop_joint name="${prefix}_finger_1" xyz="${x} ${y} ${z}"/>
-      <xacro:close_loop_joint name="${prefix}_finger_2" xyz="${x} ${y} ${z}"/>
+      <xacro:close_loop_joint name="${prefix}_finger_1"/>
+      <xacro:close_loop_joint name="${prefix}_finger_2"/>
     </gazebo>
-    <!-- enable mimic joints -->
-    <xacro:macro name="mimic_joint" params="name has_pid:=true">
-      <plugin name="${name}_mimic_joint_plugin" filename="libroboticsgroup_upatras_gazebo_mimic_joint_plugin.so">
-        <joint>${prefix}_joint</joint>
-        <mimicJoint>${name}</mimicJoint>
-        <multiplier>1.0</multiplier>
-        <offset>0.0</offset>
-        <sensitiveness>0.0</sensitiveness>
-        <xacro:if value="${has_pid}">
-          <hasPID/>
-          <maxEffort>${limit['effort']}</maxEffort>
-        </xacro:if>
-      </plugin>
+    <!-- tune tip's friction/collison model -->
+    <xacro:macro name="grasp_friction" params="link_name">
+      <gazebo reference="${link_name}">
+        <mu1>100</mu1>
+        <mu2>100</mu2>
+        <fdir1>0 0 1</fdir1>
+        <kp>100000</kp>
+        <kd>10</kd>
+        <collision name="${link_name}_collision">
+          <surface>
+            <friction>
+              <torsional>
+                <coefficient>0.456</coefficient>
+                <use_patch_radius>true</use_patch_radius>
+                <patch_radius>0.05</patch_radius>
+              </torsional>
+            </friction>
+          </surface>
+        </collision>
+      </gazebo>
     </xacro:macro>
-    <gazebo>
-      <xacro:mimic_joint name="${prefix}_mirror_joint"/>
-      <xacro:if value="${safety_shield}">
-        <xacro:mimic_joint name="${prefix}_finger_1_safety_shield_joint" has_pid="false"/>
-        <xacro:mimic_joint name="${prefix}_finger_2_safety_shield_joint" has_pid="false"/>
-      </xacro:if>
-    </gazebo>
+    <xacro:grasp_friction link_name="${prefix}_finger_1_flex_finger"/>
+    <xacro:grasp_friction link_name="${prefix}_finger_2_flex_finger"/>
     <!-- enable self collision -->
     <gazebo reference="${prefix}_bracket">

File: onrobot_description/urdf/onrobot_rg.transmission.xacro (robot description, xacro)
@@ -2,5 +2,5 @@
 <robot xmlns:xacro="http://ros.org/wiki/xacro">
   <xacro:macro name="rg_transmission" params="prefix hw_interface">
-    <transmission name="${prefix}_joint_trans">
+    <!-- <transmission name="${prefix}_joint_trans">
       <type>transmission_interface/SimpleTransmission</type>
       <joint name="${prefix}_joint">
@@ -11,5 +11,5 @@
         <mechanicalReduction>1</mechanicalReduction>
       </actuator>
-    </transmission>
+    </transmission> -->
   </xacro:macro>
 </robot>

File: onrobot_description/urdf/onrobot_rg.urdf.xacro (robot description, xacro)
@@ -114,5 +114,5 @@
         <xacro:_frame id="moment_arm" rpy="0.0 ${offset} 0.0"/>
         <xacro:_limit/>
-        <dynamics damping="1" friction="0"/>
+        <dynamics damping="0.5"/>
         <xacro:unless value="${is_master}">
           <mimic joint="${prefix}_joint" multiplier="1" offset="0"/>
@@ -140,5 +140,4 @@
         <xacro:_frame id="truss_arm" rpy="0.0 ${offset} 0.0"/>
         <xacro:_limit/>
-        <dynamics damping="1" friction="1"/>
         <mimic joint="${prefix}_joint" multiplier="1" offset="0"/>
       </joint>
@@ -166,5 +165,4 @@
           <xacro:_frame id="safety_shield" rpy="0.0 ${offset} 0.0"/>
           <xacro:_limit/>
-          <dynamics damping="1" friction="1"/>
           <mimic joint="${prefix}_joint" multiplier="1" offset="0"/>
         </joint>
@@ -196,5 +194,4 @@
         <xacro:_frame id="finger_tip" rpy="0.0 ${-offset} 0.0"/>
         <xacro:_limit/>
-        <dynamics damping="1" friction="1"/>
         <mimic joint="${prefix}_joint" multiplier="1" offset="0"/>
       </joint>
